File: Prototyping OTG Board/v1/Prototyping OTG Board.brd (EAGLE design)
At the start: 54.6 x 62.2 mm, 42 parts, among them U1 MCP73831, U2 TPS63001, U3 TPS61240, U4 TPS2113A.DRB, U5 TPS2113A.DRB, U6 LP38692, X1 USBSMD

Commit message: Not sure what changed to the Prototyping OTG Board...
Parts:
- moved C10 1.27 mm to (51.4, 13.3)
- moved C11 1.27 mm to (46.4, 13.3)
- moved R9 1.27 mm to (48.9, 10.8)
- moved U6 1.27 mm to (48.9, 13.3)
- moved X1 1.27 mm to (48.3, 5.08)
Changed lines of the file:
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@@
 <setting verticaltext="up"/>
 </settings>
-<grid distance="0.25" unitdist="mm" unit="mm" style="dots" multiple="2" display="yes" altdistance="0.05" altunitdist="mm" altunit="mm"/>
+<grid distance="25" unitdist="mil" unit="mil" style="dots" multiple="2" display="yes" altdistance="5" altunitdist="mil" altunit="mil"/>
 <layers>
 <layer number="1" name="Top" color="4" fill="1" visible="yes" active="yes"/>
@@
 <attribute name="NAME" x="2.794" y="14.605" size="0.8128" layer="26" ratio="15" rot="MR90"/>
 </element>
-<element name="X1" library="SparkFun" package="USB-MINIB" value="USBSMD" x="48.26" y="6.35" smashed="yes" rot="R90"/>
+<element name="X1" library="SparkFun" package="USB-MINIB" value="USBSMD" x="48.26" y="5.08" smashed="yes" rot="R90"/>
 <element name="U$3" library="SparkFun" package="BREADBOARD-MINI" value="BREADBOARDMINI" x="45.085" y="16.51" smashed="yes" rot="R90"/>
 <element name="U$24" library="samtec" package="SSW-117-22-XXX-D-VS" value="SSW-117-22-XXX-D-VS" x="5.715" y="39.37" smashed="yes" rot="R90"/>
@@
 <attribute name="NAME" x="26.289" y="12.065" size="0.8128" layer="26" font="vector" rot="MR90"/>
 </element>
-<element name="U6" library="national-semiconductor" package="LLP6" value="LP38692" x="48.895" y="14.605" smashed="yes" rot="R90">
-<attribute name="NAME" x="48.26" y="15.24" size="0.8128" layer="26" rot="MR180"/>
+<element name="U6" library="national-semiconductor" package="LLP6" value="LP38692" x="48.895" y="13.335" smashed="yes" rot="R90">
+<attribute name="NAME" x="48.26" y="13.97" size="0.8128" layer="26" rot="MR180"/>
 </element>
-<element name="R9" library=".standardparts" package="0603" value="10k" x="48.895" y="12.065" smashed="yes">
-<attribute name="NAME" x="49.53" y="11.684" size="0.8128" layer="26" font="vector" rot="MR0"/>
+<element name="R9" library=".standardparts" package="0603" value="10k" x="48.895" y="10.795" smashed="yes">
+<attribute name="NAME" x="49.53" y="10.414" size="0.8128" layer="26" font="vector" rot="MR0"/>
 </element>
-<element name="C10" library=".standardparts" package="0603" value="4.7uF" x="51.435" y="14.605" smashed="yes" rot="R270">
-<attribute name="NAME" x="51.816" y="15.621" size="0.8128" layer="26" font="vector" rot="MR270"/>
+<element name="C10" library=".standardparts" package="0603" value="4.7uF" x="51.435" y="13.335" smashed="yes" rot="R270">
+<attribute name="NAME" x="51.816" y="14.351" size="0.8128" layer="26" font="vector" rot="MR270"/>
 </element>
-<element name="C11" library=".standardparts" package="0603" value="4.7uF" x="46.355" y="14.605" smashed="yes" rot="R90">
-<attribute name="NAME" x="46.736" y="15.621" size="0.8128" layer="26" font="vector" rot="MR270"/>
+<element name="C11" library=".standardparts" package="0603" value="4.7uF" x="46.355" y="13.335" smashed="yes" rot="R90">
+<attribute name="NAME" x="46.736" y="14.351" size="0.8128" layer="26" font="vector" rot="MR270"/>
 </element>
 <element name="R11" library=".standardparts" package="0603" value="10k" x="12.7" y="7.366" smashed="yes" rot="R180">
@@
 <contactref element="U4" pad="8"/>
 <contactref element="C9" pad="2"/>
-<contactref element="U6" pad="4"/>
-<contactref element="U6" pad="5"/>
-<contactref element="C11" pad="2"/>
 <contactref element="U2" pad="10"/>
 <contactref element="U2" pad="1"/>
 <contactref element="C2" pad="2"/>
 <contactref element="ON/OFF" pad="2"/>
-<wire x1="47.495" y1="14.605" x2="47.495" y2="15.555" width="0" layer="19" extent="1-1"/>
-<wire x1="46.355" y1="15.38" x2="47.495" y2="15.555" width="0" layer="19" extent="1-1"/>
-<wire x1="37.76" y1="14.81" x2="46.355" y2="15.38" width="0" layer="19" extent="1-1"/>
+<contactref element="U6" pad="5"/>
+<contactref element="C11" pad="2"/>
+<contactref element="U6" pad="4"/>
+<wire x1="47.495" y1="14.285" x2="47.495" y2="13.335" width="0" layer="19" extent="1-1"/>
+<wire x1="46.355" y1="14.11" x2="47.495" y2="14.285" width="0" layer="19" extent="1-1"/>
+<wire x1="37.76" y1="14.81" x2="46.355" y2="14.11" width="0" layer="19" extent="1-1"/>
 <wire x1="35.56" y1="14.11" x2="37.76" y2="14.81" width="0" layer="19" extent="1-1"/>
 <wire x1="15.367" y1="10.935" x2="35.56" y2="14.11" width="0" layer="19" extent="1-1"/>
@@
 <contactref element="C10" pad="2"/>
 <contactref element="R9" pad="2"/>
-<wire x1="50.295" y1="13.655" x2="50.295" y2="15.555" width="0" layer="19" extent="1-1"/>
-<wire x1="51.435" y1="13.83" x2="50.295" y2="13.655" width="0" layer="19" extent="1-1"/>
-<wire x1="49.67" y1="12.065" x2="50.295" y2="13.655" width="0" layer="19" extent="1-1"/>
-<wire x1="47.495" y1="13.655" x2="49.67" y2="12.065" width="0" layer="19" extent="1-1"/>
-<wire x1="46.66" y1="8.85" x2="49.67" y2="12.065" width="0" layer="19" extent="1-1"/>
-<wire x1="30.17" y1="11.225" x2="46.66" y2="8.85" width="0" layer="19" extent="1-1"/>
+<wire x1="50.295" y1="12.385" x2="50.295" y2="14.285" width="0" layer="19" extent="1-1"/>
+<wire x1="51.435" y1="12.56" x2="50.295" y2="12.385" width="0" layer="19" extent="1-1"/>
+<wire x1="49.67" y1="10.795" x2="50.295" y2="12.385" width="0" layer="19" extent="1-1"/>
+<wire x1="47.495" y1="12.385" x2="49.67" y2="10.795" width="0" layer="19" extent="1-1"/>
+<wire x1="46.66" y1="7.58" x2="49.67" y2="10.795" width="0" layer="19" extent="1-1"/>
+<wire x1="30.17" y1="11.225" x2="46.66" y2="7.58" width="0" layer="19" extent="1-1"/>
 <wire x1="28.87" y1="14.175" x2="30.17" y2="11.225" width="0" layer="19" extent="1-1"/>
 <wire x1="29.07" y1="15.875" x2="28.87" y2="14.175" width="0" layer="19" extent="1-1"/>
