File: Prototyping OTG Board/v1/Prototyping OTG Board.sch (EAGLE design)
At the start: 42 parts, among them U1 MCP73831, U2 TPS63001, U3 TPS61240, U4 TPS2113A.DRB, U5 TPS2113A.DRB, U6 LP38692, X1 USBSMD

Commit message: Not sure what changed to the Prototyping OTG Board...
Other:
- note added: "Power Control"
- moved on the sheet: 3.3V.EN, 5V.EN, C11, ON/OFF, R10, R2, R4, SELECT
