File: TI/Robotics Booster Pack/Robotics Booster Pack.sch (EAGLE design)
At the start: 117 parts, among them U1 DRV8800, U10 74LVTH125.RGY, U11 SCHA4B0400, U12 BLUETOOTH-RN41", U13 XBEE-1XBEE-1_LOCK, U14 FDMA3028N, U2 DRV8800, U3 DRV8800, U4 DRV8800, U5 TPS5331[8/9].DQP, U6 TPS62082.DSG, U7 PCA9557.RGV, U8 MPU-6050, U9 INA220.DGS

Commit message: Making progress on PCB re-layout. Moved some pins around to make routing _much_ easier, along with the added improvements.
Parts:
- removed H21: 1X2.PTS, phoenixcontact:1X2.PTS.PLUG
- removed H8: 1X3, headers(.1in):1X3
- removed J5, J6, J7, J8: (no value), solderjumper:SOLDERJUMPER.2.LRG
- removed U$9: 2X4, headers(.1in):2X4
- removed U14: FDMA3028N, freescale:FDMA1024NZ
- added D3, D4: CDBMT2100-HF, comchip:CDBMT____-HF
- added J1: 1X2.PTS, phoenixcontact:1X2.PTS.PLUG
- added J3: (no value), solderjumper:SOLDERJUMPER.2.LRG
- added Q1: (no value), fairchild:FDMA
- added U$6: 1X4, headers(.1in):1X4
- D1, D2: value (none) -> CDBMT2100-HF; device nxp:DIODE[SCHOTKY]-SOD123W -> comchip:CDBMT____-HF
- R1: value 178k -> 1u; device standardparts:RESISTOR.0603 -> vishay:RESISTOR.WSK
- R3: value 1u -> 178k; device vishay:RESISTOR.WSK -> standardparts:RESISTOR.0603
- U1: value DRV8800 -> TPS5331[8/9].DQP; device packages(ti):DRV8800.RTY -> packages(ti):TPS5331[8/9].DQP
- U2: value DRV8800 -> TPS62082.DSG; device packages(ti):DRV8800.RTY -> packages(ti):TPS6208X.DSG
- U5: value TPS5331[8/9].DQP -> DRV8800; device packages(ti):TPS5331[8/9].DQP -> packages(ti):DRV8800.RTY
- U6: value TPS62082.DSG -> DRV8800; device packages(ti):TPS6208X.DSG -> packages(ti):DRV8800.RTY
Connections:
- removed net N$16: H8.1, H8.2, H8.3
- removed net VIN: C2.1, D2.2, U$8.VBUS, U6.VIN
- new net VFET: D3.1, D4.1, H7.1, H7.2, H7.3, J3.1
- new net VSERVO: C12.2, C14.+, C39.+, D2.2, H2.1, H2.2, H2.3, H2.4, H2.5, H2.6, H22.1, L1.2, R15.1
- net 3.3V: now also C1.1, R3.2, U$6.1, U2.VOS; no longer C35.1, R1.2, U$9.1, U$9.2, U6.VOS
- net 3.3V.PG: now also R3.1, U2.PG; no longer R1.1, U6.PG
- net 5.0V: now also C2.1, U$8.VBUS, U2.VIN; no longer C12.2, C14.+, C39.+, H2.1, H2.2, H2.3, H2.4, H2.5, H2.6, H22.1, L1.2, R15.1
- net 5V.PG: now also U1.PGOOD, U2.EN; no longer U5.PGOOD, U6.EN
- net FET0.D: now also D3.2, Q1.A.D; no longer U14G$1.D
- net FET0.G: now also Q1.A.G; no longer U14G$1.G
- net FET1.D: now also D4.2, H9.3, Q1.B.D; no longer H9.2, U14G$2.D
- net FET1.G: now also Q1.B.G; no longer U14G$2.G
- net GND: now also C1.2, D1.2, H9.2, J1.2, Q1.A.S, Q1.B.S, U$6.4, U2.MODE, U5.SENSE, U6.SENSE; no longer C35.2, D1.1, H21.2, H7.1, H7.2, H7.3, U$9.7, U$9.8, U1.SENSE, U14G$1.S, U14G$2.S, U2.SENSE, U6.MODE
- net I2C.SCL: now also U$6.3; no longer U$9.5, U$9.6
- net I2C.SDA: now also U$6.2; no longer U$9.3, U$9.4
- net M.EN: now also U5.!SLEEP, U6.!SLEEP; no longer U1.!SLEEP, U2.!SLEEP
- net M.MODE: now also U5.MODE, U6.MODE; no longer U1.MODE, U2.MODE
- net M0+: now also U5.OUT+; no longer U1.OUT+
- net M0-: now also U5.OUT-; no longer U1.OUT-
- net M0.DIR: now also U$8.PF0, U5.ENABLE; no longer J6.1, U$8.PC4, U1.ENABLE
- net M0.SPD: now also U$8.PA7, U5.PHASE; no longer J5.1, U$8.PD0, U1.PHASE
- net M1+: now also U6.OUT+; no longer U2.OUT+
- net M1-: now also U6.OUT-; no longer U2.OUT-
- net M1.DIR: now also U$8.PF4, U6.ENABLE; no longer J6.2, U$8.PC7, U2.ENABLE
- net M1.SPD: now also U$8.PA6, U6.PHASE; no longer J5.2, U$8.PD1, U2.PHASE
- net M2.DIR: now also U$8.PC4; no longer J8.1, U$8.PF0
- net M2.SPD: now also U$8.PD1; no longer J7.1, U$8.PA6
- net M3.DIR: now also U$8.PC7; no longer J8.2, U$8.PF4
- net M3.SPD: now also U$8.PD0; no longer J7.2, U$8.PA7
- net N$10: now also U1.FB; no longer U5.FB
- net N$12: now also U2.SW; no longer U6.SW
- net N$13: now also U5.CP2; no longer U1.CP2
- net N$15: now also C35.2, U1.LL; no longer C1.2, U5.LL
- net N$18: now also U5.VCP; no longer U1.VCP
- net N$19: now also U6.VCP; no longer U2.VCP
- net N$2: now also C35.1, U1.VBST; no longer C1.1, U5.VBST
- net N$22: now also D1.1, J1.1, R1.1; no longer D1.2, H21.1, R3.1
- net N$25: now also U6.CP2; no longer U2.CP2
- net N$3: now also U1.MODE; no longer U5.MODE
- net N$38: now also U5.CP1; no longer U1.CP1
- net N$39: now also U6.CP1; no longer U2.CP1
- net N$4: now also U1.VREG; no longer U5.VREG
- net N$5: now also U1.TRIP; no longer U5.TRIP
- net N$8: now also U1.EN; no longer U5.EN
- net VBAT: now also J3.2, R1.2, U1.VDD, U1.VIN, U5.VMOT, U6.VMOT; no longer H9.3, R3.2, U1.VMOT, U2.VMOT, U5.VDD, U5.VIN
Other:
- note added: "NOTES: - Consider PCA9539 - Individual Motor EN control - Might not be enough routing space to begin with - Tweak 5v circuit value to output 5.5v - Too much voltage sag at lower voltages - Change headers to Samtec Parts - Update Rn-41/2 Footprint - Remove VBAT GND headers - Change VBAT <> VIN header to SMD Jumper"
- note removed: "NOTES: - Move I2C and UART 50mil to left - Connect BT.RESET to IO Expander"
- moved on the sheet: C1, C10, C11, C12, C13, C14, C15, C2, C20, C22, C3, C32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

Commit message: Replaced 5v regulator circuit with TPS5450 Added more power options in the form of SMD Jumpers Added IO Expander-controlled Servo FET Swapped positions of XBee and extra IO/FETs to make routing simpler Connected 5v and 3.3v from BoosterPack to Launchpad Added header to connect to UART0 (Wireless programming/debugging)
Parts:
- removed C10: 4.7uF, standardparts:CAPACITOR.0805
- removed C11: 1uF, standardparts:CAPACITOR.0603
- removed C12, C35: .1uF, standardparts:CAPACITOR.0603
- removed C13: 1nF, standardparts:CAPACITOR.0603
- removed C14: 100uF, microbuilder:CAP_ELECTROLYTICPANASONIC_D
- removed H22, H26: 1X2, headers(.1in):1X2
- removed L1: 2.2uH, coilcraft:INDUCTOR.XAL6030
- removed R10: 1k, standardparts:RESISTOR.0603
- removed R11, R12: 100k, standardparts:RESISTOR.0603
- removed R13: 191k, standardparts:RESISTOR.0603
- removed R14: 2.55k, standardparts:RESISTOR.0603
- removed R15: 76.8k, standardparts:RESISTOR.0603
- removed R16: 10k, standardparts:RESISTOR.0603
- removed R8: 200k, standardparts:RESISTOR.0603
- removed R9: 86.6k, standardparts:RESISTOR.0603
- removed RXI, TXO: (no value), solderjumper:SOLDERJUMPER.3.LRG.12
- added C40: 330uF, microbuilder:CAP_ELECTROLYTICPANASONIC_D
- added C41: 10nF, standardparts:CAPACITOR.0603
- added C42: 10uF, standardparts:CAPACITOR.1206
- added D5: CDBMT2100-HF, comchip:CDBMT____-HF
- added D6: CDBC5XXX-G, comchip:CDBC5XXX-G
- added J4: (no value), solderjumper:SOLDERJUMPER.3.LRG.12
- added J6, J7: (no value), solderjumper:SOLDERJUMPER.3.LRG
- added J9: (no value), solderjumper:SOLDERJUMPER.2.LRG.PASTE
- added L3: INDUCTOR.XAL6060, coilcraft:INDUCTOR.XAL6060
- added Q2: (no value), fairchild:FDMA
- added R17: 10k, standardparts:RESISTOR.0603
- added R18: 2.87k, standardparts:RESISTOR.0603
- added U$15: 1X2, headers(.1in):1X2
- added U14: TPS54X0, packages(ti):TPS54X0
- C39: value 100uF -> 220uF
- C9: value 22uF -> 100uF; device standardparts:CAPACITOR.1206 -> microbuilder:CAP_ELECTROLYTICPANASONIC_D
- H1, H2, H4, H5: value 1X6 -> 1X7; device headers(.1in):1X6 -> headers(.1in):1X7
- U1: value TPS5331[8/9].DQP -> TS3A44159.RGT; device packages(ti):TPS5331[8/9].DQP -> packages(ti):TS3A44159.RGT
Connections:
- removed net N$23: LED3.2, RA1.2.2
- removed net N$30: LED1.1, RA1.4.2
- removed net N$31: LED2.1, RA1.3.2
- removed net N$46: LED7.2, RA2.2.1
- removed net N$47: LED6.2, RA2.3.1
- removed net N$48: LED5.2, RA2.4.1
- removed net UART.RXI: RXI.2, U$8.PB0, U10.2A
- removed net UART.TXO: TXO.2, U$8.PB1, U10.1A
- new net N$16: J4.2, Q2.A.D, Q2.B.D
- new net N$33: C41.1, U14.BOOT
- new net N$34: C41.2, D6.1, L3.1, U14.PH
- new net N$35: R17.1, R18.2, U14.VSENSE
- new net SRVO.EN: Q2.A.G, Q2.B.G, U7.P7
- new net UART0.RXI: U1.IN2
- new net UART0.TXO: U1.IN1
- new net UART1.RXI: U$8.PB0, U1.IN3, U10.2A
- new net UART1.TXO: U$8.PB1, U1.EN3,4, U10.1A
- net 3.3V: now also J6.1, J7.1, J9.1, U$8.3.3V, U1.VCC; no longer C34.+, H26.1, H5.1, H5.2, H5.3, H5.4, H5.5, H5.6
- net 5.0V: now also C40.+, D2.2, J4.3, L3.2, R17.2; no longer D2.1, U$8.VBUS
- net 5V.PG: no longer R11.2, U1.PGOOD
- net AD0: now also H6.1, U$8.PD2; no longer H6.6, U$8.PE3
- net AD1: now also H6.2, U$8.PD3; no longer H6.5, U$8.PE2
- net AD2: now also H6.3, U$8.PE0; no longer H6.4, U$8.PE1
- net AD3: now also H6.4, U$8.PE1; no longer H6.3, U$8.PE0
- net AD4: now also H6.5, U$8.PE2; no longer H6.2, U$8.PD3
- net AD5: now also H6.6, U$8.PE3; no longer H6.1, U$8.PD2
- net BT.RXI: now also U1.O2, U1.O4; no longer RXI.1
- net BT.TXO: now also U1.O1, U1.O3; no longer TXO.1
- net FET0.G: now also U7.P0; no longer U7.P4
- net FET1.G: now also U7.P1; no longer U7.P5
- net GND: now also C40.-, C42.2, D5.2, D6.2, H1.7, H4.7, J6.3, J7.3, R18.1, U14.GND; no longer C10.2, C11.1, C14.-, C9.2, H22.2, H26.2, R12.1, R13.2, R16.2, R9.1
- net IO0: now also U7.P5; no longer U7.P0
- net IO1: now also U7.P4; no longer U7.P1
- net IO2: now also U7.P3; no longer U7.P2
- net IO3: now also U7.P2; no longer U7.P3
- net M.EN: now also U7.P6; no longer U7.P7
- net N$1: now also D2.1, U$8.VBUS; no longer U$8.3.3V
- net N$10: now also LED2.1, RA1.2.2; no longer C13.1, R15.2, R16.1, U1.FB
- net N$11: now also LED1.1, RA1.1.2; no longer R10.1, R8.2, R9.2
- net N$14: now also LED8.2, RA2.4.1; no longer C12.1, C13.2, R14.2
- net N$15: now also LED6.2, RA2.2.1; no longer C35.2, L1.1, R14.1, U1.LL
- net N$17: now also LED5.2, RA2.1.1; no longer LED4.2, RA1.1.2
- net N$2: now also J6.2, U1.EN1,2; no longer C35.1, U1.VBST
- net N$22: now also C9.+
- net N$3: now also J7.2, U1.IN4; no longer R12.2, U1.MODE
- net N$4: now also C34.+, H5.1, H5.2, H5.3, H5.4, H5.5, H5.6, H5.7, J9.2; no longer C11.2, R11.1, U1.VREG
- net N$5: now also LED4.2, RA1.4.2; no longer R13.1, U1.TRIP
- net N$8: now also LED3.2, RA1.3.2; no longer R10.2, U1.EN
- net N$9: now also LED7.2, RA2.3.1; no longer LED8.2, RA2.1.1
- net VBAT: now also C42.1, J4.1, U14.VIN; no longer C10.1, C9.1, R8.1, U1.VDD, U1.VIN
- net VSERVO: now also D5.1, H2.7, Q2.A.S, Q2.B.S; no longer C12.2, C14.+, D2.2, H22.1, L1.2, R15.1
- net XBEE.RXI: now also U1.!O2, U1.!O4; no longer RXI.3
- net XBEE.TXO: now also U1.!O1, U1.!O3; no longer TXO.3
Other:
- note added: "NOTES: - Tweak 5v circuit value to output 5.5v - Too much voltage sag at lower voltages - Double Check: Confirm diode isn't droppong voltage too low/cause wasn't because of 2S Lipo - Change headers to Samtec Parts - Update Rn-41/2 Footprint - Add Power/En to BT and XBee"
- note removed: "NOTES: - Consider PCA9539 - Individual Motor EN control - Might not be enough routing space to begin with - Tweak 5v circuit value to output 5.5v - Too much voltage sag at lower voltages - Change headers to Samtec Parts - Update Rn-41/2 Footprint - Remove VBAT GND headers - Change VBAT <> VIN header to SMD Jumper"
- moved on the sheet: C1, C34, C38, C39, D1, D2, H3, H6, J1, LED5, LED6, R1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
